Commit message: Initial commit

File: src/cad/CAD_ASR_WITH_OMNI.urdf (robot description, URDF)
Before this commit: robot CAD_ASR_WITH_OMNI, 7 links, 6 joints
Links:
- link base_link: geometry collision box size=0.3 0.3 0.1; visual mesh filename=package://CAD_ASR_WITH_OMNI_LENGKAP/meshes/base_link.stl scale=0.001 0.001 0.001
- link wheel_back_left: geometry collision cylinder length=0.05 radius=0.04; visual mesh filename=package://CAD_ASR_WITH_OMNI_LENGKAP/meshes/wheel_back_left.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 scale=0.001 0.001 0.001
- link wheel_back_right: geometry collision cylinder length=0.05 radius=0.04; visual mesh filename=package://CAD_ASR_WITH_OMNI_LENGKAP/meshes/wheel_back_right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 scale=0.001 0.001 0.001
- link wheel_front: geometry collision cylinder length=0.05 radius=0.04; visual mesh filename=package://CAD_ASR_WITH_OMNI_LENGKAP/meshes/wheel_front.stl scale=0.001 0.001 0.001
Joints:
- joint base_link_wheel_back_left_to_base_link: origin xyz=-0.2202118253752416 0.055999996502206474 0.10821198883837659 rpy=9.316995221376523e-16 1.061160185212551 -3.1415926535897922 -> xyz=-0.070 0.054 -0.150 rpy=0 0.500000 0
- joint base_link_wheel_back_right_to_base_link: origin xyz=0.21735475462475834 0.05599896650220654 0.11366768883837633 rpy=-6.405199662469398e-17 -1.043706892692612 -3.141592653589793 -> xyz=-0.073 0.054 0.150 rpy=3.141593 0.541593 3.141593
- joint base_link_wheel_front_to_base_link: origin xyz=8.51446247581933e-05 0.055999996502206405 -0.27189263116162354 rpy=3.141592653589793 5.551115123125781e-16 1.1405732311823952e-16 -> xyz=0.270 0.054 0.000 rpy=0 1.570800 0
- joint thermal_joint: origin xyz=0.169931 0.660016 0.0 rpy=0 0 -0.26 -> xyz=0.169931 0.660016 0.0 rpy=0 0 -0.52
